Commit message: update code for realtime run

File: src/simu_visual/urdf/delta_robot.urdf (robot description, URDF)
Before this commit: robot Delta_robot, 13 links, 12 joints
Links:
- link actuador: geometry visual cylinder length=0.001 radius=0.025
- link barra1_b: geometry visual box size=0.465 0.003 0.003
- link barra2_b: geometry visual box size=0.465 0.003 0.003
- link barra3_b: geometry visual box size=0.465 0.003 0.003
- link base_link: geometry visual cylinder length=0.005 radius=0.1055
- link brazo1: geometry visual box size=0.200 0.003 0.003
- link brazo2: geometry visual box size=0.200 0.003 0.003
- link brazo3: geometry visual box size=0.200 0.003 0.003
Joints:
- joint base_brazo1: origin xyz=-0.181865335 0.105 0 rpy=0 0 2.61799 -> xyz=-0.0913656801 0.05275 0 rpy=0 0 2.61799
- joint base_brazo2: origin xyz=0 -0.210 0 rpy=0 0 -1.57075 -> xyz=0 -0.1055 0 rpy=0 0 -1.57075
- joint base_brazo3: origin xyz=0.181865335 0.105 0 rpy=0 0 0.523599 -> xyz=0.0913656801 0.05275 0 rpy=0 0 0.523599
- joint codo1_a: origin xyz=0.620 0 0 rpy=0 0 0 -> xyz=0.200 0 0 rpy=0 0 0
- joint codo2_a: origin xyz=0.620 0 0 rpy=0 0 0 -> xyz=0.200 0 0 rpy=0 0 0
- joint codo3_a: origin xyz=0.620 0 0 rpy=0 0 0 -> xyz=0.200 0 0 rpy=0 0 0
