Commit message: Refactor delta robot package and fix RViz TF/end-effector mapping.
Modernize CMake and nodes, add joint_state_config and unit tests, fix URDF
prismatic chain and launch/RViz setup so the TCP and TF tree display correctly.

Co-authored-by: Cursor <cursoragent@cursor.com>

File: src/urdf/delta_robot.urdf (robot description, URDF)
Before this commit: robot Delta_robot, 14 links, 13 joints
Links:
- link actuador: geometry visual cylinder length=0.02 radius=0.012
Joints:
- joint act_x: axis (none) -> 1 0 0; limit lower=-1 upper=1 effort=100.0 velocity=0.5 -> lower=-0.6 upper=0.6 effort=100.0 velocity=0.5
- joint act_y: axis (none) -> 0 1 0; limit lower=-1 upper=1 effort=100.0 velocity=0.5 -> lower=-0.6 upper=0.6 effort=100.0 velocity=0.5; origin xyz=0 0 0 rpy=0 0 1.57075 -> xyz=0 0 0 rpy=0 0 0
- joint act_z: axis (none) -> 0 0 1; limit lower=0 upper=1 effort=100.0 velocity=0.5 -> lower=-0.6 upper=0.2 effort=100.0 velocity=0.5; origin xyz=0 0 0 rpy=0 -1.57075 0 -> xyz=0 0 0 rpy=0 0 0
- joint gripper: limit lower=0 upper=1 effort=100.0 velocity=0.5 -> (none); origin xyz=0 0 0 rpy=0 -1.57075 0 -> xyz=0 0 0 rpy=0 0 0
