Commit message: add initial_pose_publisher.py

File: src/urdf/delta_robot.urdf (robot description, URDF)
Before this commit: robot Delta_robot, 14 links, 13 joints
Links:
- link brazo1: geometry visual box size=0.200 0.01 0.01
- link brazo2: geometry visual box size=0.200 0.01 0.01
- link brazo3: geometry visual box size=0.200 0.01 0.01

Commit message: Add GUI drawing command interface

File: src/urdf/delta_robot.urdf (robot description, URDF)
Before this commit: robot delta_robot, 14 links, 13 joints
Links:
- link actuador: geometry visual cylinder length=0.002 radius=0.03
